Commit message: changes in the urdf, added grasp_ee link , and separate node for directly publishing the object xyz pose which is working

File: ros2_ws/src/ur10e_robot_description/urdf/ur10e_robotiq.urdf (robot description, URDF)
Before this commit: robot ur10e, 25 links, 24 joints
Links:
- link left_inner_finger_pad: mass None -> 0.01
- link right_inner_finger_pad: mass None -> 0.01

File: ros2_ws/src/ur10e_robot_description/urdf/ur10e_robotiq.urdf.xacro (robot description, xacro)
@@ -70,4 +70,18 @@
     <origin xyz="0 0 0" rpy="0 0 0"/>
   </xacro:robotiq_gripper>
+  <!-- ===================== Grasp TCP frame ===================== -->
+  <!-- A massless frame on the gripper approach axis (tool0 +Z), at the depth of the
+       finger pads. It is the MoveIt group tip (see ur10e.srdf), so a Cartesian goal
+       is reached by the GRASP POINT, not the wrist flange — you can command an
+       object's position directly, with no manual tool offset in any node.
+       Tune 0.16 to your true grasp depth once the robot is loaded:
+         ros2 run tf2_ros tf2_echo tool0 left_inner_finger_pad    # read z
+         ros2 run tf2_ros tf2_echo tool0 right_inner_finger_pad   # read z; average -->
+  <link name="${tf_prefix}grasp_tcp"/>
+  <joint name="${tf_prefix}tool0-grasp_tcp" type="fixed">
+    <parent link="${tf_prefix}tool0"/>
+    <child link="${tf_prefix}grasp_tcp"/>
+    <origin xyz="0 0 0.16" rpy="0 0 0"/>
+  </joint>
   <!-- ===================== Single Isaac ros2_control system (arm + gripper) ===================== -->
   <!-- One system for ALL driven joints (6 arm + finger_joint). This makes the
